Commit message: Changing the joint type

File: hidex_description/urdf/hidex.urdf.xacro (robot description, xacro)
@@ -1,4 +1,4 @@
 <?xml version="1.0"?>
-<robot name="Peeler" xmlns:xacro="http://www.ros.org/wiki/xacro">
+<robot name="Hidex" xmlns:xacro="http://www.ros.org/wiki/xacro">
   <!-- Links -->
   <xacro:macro name="Hidex" params = "prefix">
@@ -7,5 +7,5 @@
       <origin xyz="0 0 0" rpy="0 0 0"/>
       <geometry>
-        <mesh filename="package://pf400_description/meshes/hidex_body.STL" scale="0.001 0.001 0.001"/>
+        <mesh filename="package://hidex_description/meshes/hidex_body.STL" scale="0.001 0.001 0.001"/>
       </geometry>
       <material name="black"/>
@@ -13,5 +13,5 @@
     <collision>
       <geometry>
-        <mesh filename="package://pf400_description/meshes/hidex_body.STL" scale="0.001 0.001 0.001"/>
+        <mesh filename="package://hidex_description/meshes/hidex_body.STL" scale="0.001 0.001 0.001"/>
       </geometry>
       <origin xyz="0 0 0" rpy="0 0 0"/>
@@ -22,5 +22,5 @@
       <origin xyz="0 0 0" rpy="0 0 0"/>
       <geometry>
-        <mesh filename="package://pf400_description/meshes/hidex_plate.STL" scale="0.001 0.001 0.001"/>
+        <mesh filename="package://hidex_description/meshes/hidex_plate.STL" scale="0.001 0.001 0.001"/>
       </geometry>
       <material name="aluminum"/>
@@ -28,5 +28,5 @@
     <collision>
       <geometry>
-        <mesh filename="package://pf400_description/meshes/hidex_plate.STL" scale="0.001 0.001 0.001"/>
+        <mesh filename="package://hidex_description/meshes/hidex_plate.STL" scale="0.001 0.001 0.001"/>
       </geometry>
       <origin xyz="0 0 0" rpy="0 0 0"/>
@@ -34,5 +34,5 @@
   </link>
   <!-- Joints -->
-  <joint name="Hidex_Plate_Joint" type="fixed">
+  <joint name="Hidex_Plate_Joint" type="prismatic">
     <parent link="${prefix}hidex_body"/>
     <child link="${prefix}hidex_plate"/>

Commit message: Update

File: hidex_description/urdf/hidex.urdf.xacro (robot description, xacro)
@@ -3,5 +3,5 @@
   <!-- Links -->
   <xacro:macro name="Hidex" params = "prefix">
-    <link name="${prefix}hidex_body">
+  <link name="${prefix}hidex_body">
     <visual>
       <origin xyz="0 0 0" rpy="0 0 0"/>
